Commit message: added inertia and collision to the urdf file

File: robotic_arm_description/urdf/arm.urdf.xacro (robot description, xacro)
@@ -4,6 +4,16 @@
     <xacro:property name="effort" value="30.0" />
     <xacro:property name="velocity" value="10.0" />
+    <xacro:macro name="default_inertial" params="mass">
+        <inertial>
+            <origin xyz="0 0 0" rpy="0 0 0"/>
+            <mass value="${mass}" />
+            <inertia ixx="1.0" ixy="0.0" ixz="0.0"
+                     iyy="1.0" iyz="0.0"
+                     izz="1.0" />
+        </inertial>
+    </xacro:macro>
     <link name="world"/>
     <link name="base_link">
+        <xacro:default_inertial mass="1.0"/>
         <visual>
             <origin rpy="0 0 0" xyz="-0.5 -0.5 0" />
@@ -12,4 +22,10 @@
             </geometry>
         </visual>
+        <collision>
+            <origin rpy="0 0 0" xyz="-0.5 -0.5 0"/>
+            <geometry>
+                <mesh filename="package://arduinobot_description/meshes/basement.STL" scale="0.01 0.01 0.01"/>
+            </geometry>
+        </collision>
     </link>
     <joint name="virtual_joint" type="fixed">
@@ -19,4 +35,5 @@
     </joint>
     <link name="base_plate">
+        <xacro:default_inertial mass="0.1"/>
         <visual>
             <origin rpy="0 0 0" xyz="-0.39 -0.39 -0.56" />
@@ -25,4 +42,10 @@
             </geometry>
         </visual>
+        <collision>
+            <origin rpy="0 0 0" xyz="-0.39 -0.39 -0.56"/>
+            <geometry>
+                <mesh filename="package://arduinobot_description/meshes/base_plate.STL" scale="0.01 0.01 0.01"/>
+            </geometry>
+        </collision>
     </link>
     <joint name="joint_1" type="revolute">
@@ -34,4 +57,5 @@
     </joint>
     <link name="forward_drive_arm">
+        <xacro:default_inertial mass="0.1"/>
         <visual>
             <origin rpy="0 -${PI/2} ${PI/2}" xyz="0.19 0.06 -0.08" />
@@ -40,4 +64,10 @@
             </geometry>
         </visual>
+        <collision>
+            <origin rpy=" 0 -${PI / 2} ${PI / 2}" xyz="0.19 0.06 -0.08"/>
+            <geometry>
+                <mesh filename="package://arduinobot_description/meshes/forward_drive_arm.STL" scale="0.01 0.01 0.01"/>
+            </geometry>
+        </collision>
     </link>
     <joint name="joint_2" type="revolute">
@@ -49,4 +79,5 @@
     </joint>
     <link name="horizontal_arm">
+        <xacro:default_inertial mass="0.1"/>
         <visual>
             <origin rpy="${PI/2} 0 ${PI/2}" xyz="-0.03 -0.4 -0.06" />
@@ -55,4 +86,10 @@
             </geometry>
         </visual>
+        <collision>
+            <origin rpy="${PI / 2} 0 ${PI / 2}" xyz="-0.03 -0.4 -0.06"/>
+            <geometry>
+                <mesh filename="package://arduinobot_description/meshes/horizontal_arm.STL" scale="0.01 0.01 0.01"/>
+            </geometry>
+        </collision>
     </link>
     <joint name="joint_3" type="revolute">
@@ -64,4 +101,5 @@
     </joint>
     <link name="claw_support">
+        <xacro:default_inertial mass="0.1"/>
         <visual>
             <origin rpy="0 0 ${PI/2}" xyz="0 -0.05 -0.15" />
@@ -70,4 +108,10 @@
             </geometry>
         </visual>
+        <collision>
+            <origin rpy="0 0 ${PI / 2}" xyz="0 -0.05 -0.15"/>
+            <geometry>
+                <mesh filename="package://arduinobot_description/meshes/claw_support.STL" scale="0.01 0.01 0.01"/>
+            </geometry>
+        </collision>
     </link>
     <joint name="horizontal_arm_to_claw_support" type="fixed">
@@ -77,4 +121,5 @@
     </joint>
      <link name="gripper_right">
+        <xacro:default_inertial mass="0.1"/>
         <visual>
             <origin rpy="0 0 -${PI/2}" xyz="-0.1 0.5 -0.1" />
@@ -83,6 +128,13 @@
             </geometry>
         </visual>
+        <collision>
+            <origin rpy="0 0 -${PI / 2}" xyz="-0.1 0.50 -0.1"/>
+            <geometry>
+                <mesh filename="package://arduinobot_description/meshes/right_finger.STL" scale="0.01 0.01 0.01"/>
+            </geometry>
+        </collision>
     </link>
      <link name="gripper_left">
+        <xacro:default_inertial mass="0.1"/>
         <visual>
             <origin rpy="0 0 -${PI/2}" xyz="-0.04 0.5 -0.1" />
@@ -91,4 +143,10 @@
             </geometry>
         </visual>
+        <collision>
+            <origin rpy="0 0 -${PI / 2}" xyz="-0.04 0.50 -0.1"/>
+            <geometry>
+                <mesh filename="package://arduinobot_description/meshes/left_finger.STL" scale="0.01 0.01 0.01"/>
+            </geometry>
+        </collision>
     </link>
     <joint name="joint_4" type="revolute">

Commit message: added urdf modification

File: robotic_arm_description/urdf/arm.urdf.xacro (robot description, xacro)
@@ -1,5 +1,6 @@
 <?xml version="1.0"?>
-<robot xmlns:xacro="http://www.ros.org/wiki/xacro" name="roboticarm">
-    <xacro:property name="PI" value="3.14159" />
+<robot xmlns:xacro="http://www.ros.org/wiki/xacro" name="arduinobot">
+    <!-- Useful XACRO Variables (Properties) -->
+    <xacro:property name="PI" value="3.14159265359" />
     <xacro:property name="effort" value="30.0" />
     <xacro:property name="velocity" value="10.0" />
@@ -13,9 +14,10 @@
         </inertial>
     </xacro:macro>
+    <!-- Links -->
     <link name="world"/>
     <link name="base_link">
         <xacro:default_inertial mass="1.0"/>
         <visual>
-            <origin rpy="0 0 0" xyz="-0.5 -0.5 0" />
+            <origin rpy="0 0 0" xyz="-0.5 -0.5 0"/>
             <geometry>
                 <mesh filename="package://robotic_arm_description/meshes/basement.STL" scale="0.01 0.01 0.01"/>
@@ -29,15 +31,10 @@
         </collision>
     </link>
-    <joint name="virtual_joint" type="fixed">
-        <parent link="world"/>
-        <child link="base_link"/>
-        <origin rpy="0 0 0" xyz="0 0 0"/>
-    </joint>
     <link name="base_plate">
         <xacro:default_inertial mass="0.1"/>
         <visual>
-            <origin rpy="0 0 0" xyz="-0.39 -0.39 -0.56" />
+            <origin rpy="0 0 0" xyz="-0.39 -0.39 -0.56"/>
             <geometry>
-                <mesh filename="package://robotic_arm_description/meshes/base_plate.STL" scale="0.01 0.01 0.01" />
+                <mesh filename="package://robotic_arm_description/meshes/base_plate.STL" scale="0.01 0.01 0.01"/>
             </geometry>
         </visual>
@@ -49,17 +46,10 @@
         </collision>
     </link>
-    <joint name="joint_1" type="revolute">
-        <parent link="base_link" />
-        <child link="base_plate"/>
-        <axis xyz="0 0 1"/>
-        <origin rpy="0 0 0" xyz="0 0 0.307"/>
-        <limit lower="-${PI/2}" upper="${PI/2}" effort="${effort}" velocity="${velocity}"/>
-    </joint>
     <link name="forward_drive_arm">
         <xacro:default_inertial mass="0.1"/>
         <visual>
-            <origin rpy="0 -${PI/2} ${PI/2}" xyz="0.19 0.06 -0.08" />
+            <origin rpy=" 0 -${PI / 2} ${PI / 2}" xyz="0.19 0.06 -0.08"/>
             <geometry>
-                <mesh filename="package://robotic_arm_description/meshes/forward_drive_arm.STL" scale="0.01 0.01 0.01" />
+                <mesh filename="package://robotic_arm_description/meshes/forward_drive_arm.STL" scale="0.01 0.01 0.01"/>
             </geometry>
         </visual>
@@ -71,17 +61,10 @@
         </collision>
     </link>
-    <joint name="joint_2" type="revolute">
-        <parent link="base_plate" />
-        <child link="forward_drive_arm"/>
-        <axis xyz="1 0 0"/>
-        <origin rpy="0 0 0" xyz="-0.02 0 0.35"/>
-        <limit lower="-${PI/2}" upper="${PI/2}" effort="${effort}" velocity="${velocity}"/>
-    </joint>
     <link name="horizontal_arm">
         <xacro:default_inertial mass="0.1"/>
         <visual>
-            <origin rpy="${PI/2} 0 ${PI/2}" xyz="-0.03 -0.4 -0.06" />
+            <origin rpy="${PI / 2} 0 ${PI / 2}" xyz="-0.03 -0.4 -0.06"/>
             <geometry>
-                <mesh filename="package://robotic_arm_description/meshes/horizontal_arm.STL" scale="0.01 0.01 0.01" />
+                <mesh filename="package://robotic_arm_description/meshes/horizontal_arm.STL" scale="0.01 0.01 0.01"/>
             </geometry>
         </visual>
@@ -93,17 +76,10 @@
         </collision>
     </link>
-    <joint name="joint_3" type="revolute">
-        <parent link="forward_drive_arm" />
-        <child link="horizontal_arm"/>
-        <axis xyz="1 0 0"/>
-        <origin rpy="0 0 0" xyz="0 0 0.8"/>
-        <limit lower="-${PI/2}" upper="${PI/2}" effort="${effort}" velocity="${velocity}"/>
-    </joint>
     <link name="claw_support">
         <xacro:default_inertial mass="0.05"/>
         <visual>
-            <origin rpy="0 0 ${PI/2}" xyz="0 -0.05 -0.15" />
+            <origin rpy="0 0 ${PI / 2}" xyz="0 -0.05 -0.15"/>
             <geometry>
-                <mesh filename="package://robotic_arm_description/meshes/claw_support.STL" scale="0.01 0.01 0.01" />
+                <mesh filename="package://robotic_arm_description/meshes/claw_support.STL" scale="0.01 0.01 0.01"/>
             </geometry>
         </visual>
@@ -115,15 +91,10 @@
         </collision>
     </link>
-    <joint name="horizontal_arm_to_claw_support" type="fixed">
-        <parent link="horizontal_arm" />
-        <child link="claw_support"/>
-        <origin rpy="0 0 0" xyz="0 0.82 0"/>
-    </joint>
-     <link name="gripper_right">
+    <link name="gripper_right">
         <xacro:default_inertial mass="0.01"/>
         <visual>
-            <origin rpy="0 0 -${PI/2}" xyz="-0.1 0.5 -0.1" />
+            <origin rpy="0 0 -${PI / 2}" xyz="-0.1 0.50 -0.1"/>
             <geometry>
-                <mesh filename="package://robotic_arm_description/meshes/right_finger.STL" scale="0.01 0.01 0.01" />
+                <mesh filename="package://robotic_arm_description/meshes/right_finger.STL" scale="0.01 0.01 0.01"/>
             </geometry>
         </visual>
@@ -135,10 +106,10 @@
         </collision>
     </link>
-     <link name="gripper_left">
+    <link name="gripper_left">
         <xacro:default_inertial mass="0.01"/>
         <visual>
-            <origin rpy="0 0 -${PI/2}" xyz="-0.04 0.5 -0.1" />
+            <origin rpy="0 0 -${PI / 2}" xyz="-0.04 0.50 -0.1"/>
             <geometry>
-                <mesh filename="package://robotic_arm_description/meshes/left_finger.STL" scale="0.01 0.01 0.01" />
+                <mesh filename="package://robotic_arm_description/meshes/left_finger.STL" scale="0.01 0.01 0.01"/>
             </geometry>
         </visual>
@@ -150,18 +121,68 @@
         </collision>
     </link>
-    <joint name="joint_4" type="revolute">
-        <parent link="claw_support" />
-        <child link="gripper_right"/>
+    <link name="rgb_camera">
+        <visual>
+            <origin rpy="-1.57 0 -1.57" xyz="-0.1 0.125 0.15"/>
+            <geometry>
+                <mesh filename="package://robotic_arm_description/meshes/pi_camera.STL" scale="0.01 0.01 0.01"/>
+            </geometry>
+        </visual>
+    </link>
+    <!-- Joints -->
+    <joint name="virtual_joint" type="fixed">
+        <parent link="world"/>
+        <child link="base_link"/>
+        <origin xyz="0 0 0" rpy="0 0 0"/>
+    </joint>
+    <joint name ="joint_1" type="revolute">
+        <parent link="base_link"/>
+        <child link = "base_plate"/>
+        <origin xyz="0 0 0.307"/>
         <axis xyz="0 0 1"/>
-        <origin rpy="0 0 0" xyz="-0.04 0.13 -0.1"/>
-        <limit lower="-${PI/2}" upper="0.0" effort="${effort}" velocity="${velocity}"/>
+        <limit lower="-${PI / 2}" upper="${PI / 2}"
+               effort="${effort}" velocity="${velocity}"/>
     </joint>
-    <joint name="joint_5" type="revolute">
-        <parent link="claw_support" />
-        <child link="gripper_left"/>
+    <joint name ="joint_2" type="revolute">
+        <parent link="base_plate"/>
+        <child link = "forward_drive_arm"/>
+        <origin xyz="-0.02 0 0.35"/>
+        <axis xyz="1 0 0"/>
+        <limit lower="-${PI / 2}" upper="${PI / 2}"
+                effort="${effort}" velocity="${velocity}"/>
+    </joint>
+    <joint name ="joint_3" type="revolute">
+        <parent link="forward_drive_arm"/>
+        <child link = "horizontal_arm"/>
+        <origin xyz="0 0 0.8"/>
+        <axis xyz="1 0 0"/>
+        <limit lower="-${PI / 2}" upper="${PI / 2}"
+               effort="${effort}" velocity="${velocity}"/>
+    </joint>
+    <joint name ="horizontal_arm_to_claw_support" type="fixed">
+        <parent link="horizontal_arm"/>
+        <child link = "claw_support"/>
+        <origin xyz="0 0.82 0"/>
+    </joint>
+    <joint name ="joint_4" type="revolute">
+        <parent link="claw_support"/>
+        <child link = "gripper_right"/>
+        <origin xyz="-0.04 0.13 -0.1"/>
         <axis xyz="0 0 1"/>
-        <origin rpy="0 0 0" xyz="-0.22 0.13 -0.1"/>
+        <limit lower="-${PI / 2}" upper="0.0"
+               effort="${effort}" velocity="${velocity}"/>
+    </joint>
+    <joint name ="joint_5" type="revolute">
+        <parent link="claw_support"/>
+        <child link = "gripper_left"/>
+        <origin xyz="-0.22 0.13 -0.1"/>
+        <axis xyz="0 0 1"/>
+        <limit lower="0.0" upper="${PI / 2}"
+               effort="${effort}" velocity="${velocity}"/>
         <mimic joint="joint_4" multiplier="-1"/>
-        <limit lower="0.0" upper="${PI/2}" effort="${effort}" velocity="${velocity}"/>
+    </joint>
+    <joint name ="rgb_camera_joint" type="fixed">
+        <parent link="base_link"/>
+        <child link = "rgb_camera"/>
+        <origin xyz="0 0.45 0.2" rpy="0 -0.5 1.57"/>
     </joint>
 </robot>
