Commit message: Add perception, pick-and-place launch, and Gazebo world; update arm/controller configs
- Add robotic_arm_perception package with ArUco/color detection node
- Add final_build package with pick_and_place launch file
- Add pymoveit2 as tracked source (no longer a nested git repo)
- Add Gazebo world, ArUco marker model, and sensor/robot xacro files
- Rename arm.urdf.xacro to arm.xacro
- Update controller config, launch files, and CMakeLists across packages
- Remove outdated README

File: robotic_arm_description/urdf/arm.xacro (robot description, xacro)
@@ -2,8 +2,4 @@
 <robot xmlns:xacro="http://www.ros.org/wiki/xacro" name="robotic_arm">
     <xacro:arg name="is_ignition" default="true"/>
-    <!-- Include Gazebo Parameters -->
-    <xacro:include filename="$(find robotic_arm_description)/urdf/robotic_arm_gazebo.xacro" />
-    <!-- Include ros2_control Plugins -->
-    <xacro:include filename="$(find robotic_arm_description)/urdf/robotic_arm_ros2_control.xacro" />
     <!-- Useful XACRO Variables (Properties) -->
     <xacro:property name="PI" value="3.14159265359" />
@@ -89,10 +85,10 @@
             </geometry>
         </visual>
-        <collision>
+        <!-- <collision>
             <origin rpy="0 0 ${PI / 2}" xyz="0 -0.05 -0.15"/>
             <geometry>
                 <mesh filename="package://robotic_arm_description/meshes/claw_support.STL" scale="0.01 0.01 0.01"/>
             </geometry>
-        </collision>
+        </collision> -->
     </link>
     <link name="gripper_right">
@@ -123,19 +119,4 @@
             <geometry>
                 <mesh filename="package://robotic_arm_description/meshes/left_finger.STL" scale="0.01 0.01 0.01"/>
-            </geometry>
-        </collision>
-    </link>
-    <link name="rgb_camera">
-        <xacro:default_inertial mass="0.001"/>
-        <visual>
-            <origin rpy="-1.57 0 -1.57" xyz="-0.1 0.125 0.15"/>
-            <geometry>
-                <mesh filename="package://robotic_arm_description/meshes/pi_camera.STL" scale="0.01 0.01 0.01"/>
-            </geometry>
-        </visual>
-        <collision>
-            <origin rpy="-1.57 0 -1.57" xyz="-0.1 0.125 0.15"/>
-            <geometry>
-                <mesh filename="package://robotic_arm_description/meshes/pi_camera.STL" scale="0.01 0.01 0.01"/>
             </geometry>
         </collision>
@@ -193,8 +174,3 @@
         <mimic joint="joint_4" multiplier="-1"/>
     </joint>
-    <joint name ="rgb_camera_joint" type="fixed">
-        <parent link="base_link"/>
-        <child link = "rgb_camera"/>
-        <origin xyz="0 0.45 0.2" rpy="0 -0.5 1.57"/>
-    </joint>
 </robot>

File: robotic_arm_description/urdf/robotic_arm_gazebo.xacro (robot description, xacro)
@@ -1,29 +1,4 @@
 <?xml version="1.0"?>
 <robot xmlns:xacro="http://www.ros.org/wiki/xacro" name="robotic_arm">
-   <!--  <gazebo reference="rgb_camera">
-        <sensor name="camera" type="camera">
-            <always_on>true</always_on>
-            <update_rate>30.0</update_rate>
-            <visualize>true</visualize>
-            <topic>/image_raw</topic>
-            <gz_frame_id>/rgb_camera</gz_frame_id>
-            <camera name="camera">
-                <horizontal_fov>1.21126</horizontal_fov>
-                <image>
-                    <width>2304</width>
-                    <height>1296</height>
-                    <format>R8G8B8</format>
-                </image>
-                <distortion>
-                    <k1>0.0</k1>
-                    <k2>0.0</k2>
-                    <k3>0.0</k3>
-                    <p1>0.0</p1>
-                    <p2>0.0</p2>
-                    <center>0.5 0.5</center>
-                </distortion>
-            </camera>
-        </sensor>
-    </gazebo> -->
 <!-- ROS 2 Control -->
   <gazebo>
